Commit message: new sensor

File: src/b2_description/xacro/gazebo.xacro (robot description, xacro)
@@ -16,5 +16,5 @@
         <always_on>true</always_on>
         <update_rate>100</update_rate>
-        <visualize>true</visualize>
+        <visualize>false</visualize>
         <imu>
           <angular_velocity>
@@ -231,51 +231,10 @@
         <kd  value="1.0"/>
     </gazebo>
-    <gazebo reference="lidar_link">
-    <sensor name="lidar_3d" type="gpu_ray">
-        <update_rate>10</update_rate>
-        <visualize>false</visualize>
-        <ray>
-        <scan>
-            <!-- HORIZONTAL (360°) -->
-            <horizontal>
-            <samples>1800</samples>
-            <resolution>1</resolution>
-            <min_angle>-3.14159</min_angle>
-            <max_angle>3.14159</max_angle>
-            </horizontal>
-            <!-- VERTICAL (59°) -->
-            <vertical>
-            <samples>32</samples>
-            <resolution>1</resolution>
-            <min_angle>-0.9599</min_angle>   <!-- ~ -55° -->
-            <max_angle>0.2618</max_angle>    <!-- ~ +15° -->
-            </vertical>
-        </scan>
-        <range>
-            <min>0.07</min>
-            <max>100.0</max>
-            <resolution>0.01</resolution>
-        </range>
-        <noise>
-            <type>gaussian</type>
-            <mean>0.0</mean>
-            <stddev>0.007</stddev>
-        </noise>
-        </ray>
-        <!-- ROS 2 plugin -->
-        <plugin name="gazebo_ros_lidar" filename="libgazebo_ros_ray_sensor.so">
-        <ros>
-            <remapping>~/out:=rslidar_points</remapping>
-        </ros>
-        <frame_name>lidar_link</frame_name>
-        <output_type>sensor_msgs/PointCloud2</output_type>
-        </plugin>
-    </sensor>
-    </gazebo>
+    <xacro:if value="${enable_cameras}">
     <gazebo reference="f_oc_link">
     <sensor name="camera_sensor" type="camera">
         <update_rate>30</update_rate>
         <always_on>true</always_on>
-        <visualize>true</visualize>
+        <visualize>false</visualize>
         <camera>
         <horizontal_fov>1.396</horizontal_fov> <!-- ~120° -->
@@ -306,9 +265,11 @@
     </sensor>
     </gazebo>
+    </xacro:if>
+    <xacro:if value="${enable_cameras}">
     <gazebo reference="r_oc_link">
     <sensor name="camera_sensor" type="camera">
         <update_rate>30</update_rate>
         <always_on>true</always_on>
-        <visualize>true</visualize>
+        <visualize>false</visualize>
         <camera>
         <horizontal_fov>1.396</horizontal_fov> <!-- ~120° -->
@@ -339,3 +300,4 @@
     </sensor>
     </gazebo>
+    </xacro:if>
 </robot>

File: src/b2_description/xacro/robot.xacro (robot description, xacro)
@@ -1,5 +1,13 @@
 <?xml version="1.0"?>
 <robot name="b2_description" xmlns:xacro="http://www.ros.org/wiki/xacro">
+    <xacro:arg name="gpu" default="false"/>
+    <xacro:property name="gpu" value="$(arg gpu)"/>
+    <!-- false = compact 1D cloud (still has ring/time); true = full 32xN grid with NaN padding -->
+    <xacro:arg name="organize_cloud" default="false"/>
+    <xacro:property name="organize_cloud" value="$(arg organize_cloud)"/>
+    <xacro:arg name="enable_cameras" default="false"/>
+    <xacro:property name="enable_cameras" value="$(arg enable_cameras)"/>
     <xacro:include filename="$(find b2_description)/urdf/b2_description.urdf"/>
     <xacro:include filename="$(find b2_description)/xacro/gazebo.xacro"/>
+    <xacro:include filename="$(find b2_description)/xacro/lidar.xacro"/>
 </robot>

Commit message: update structure and argument

File: src/b2_description/xacro/gazebo.xacro (robot description, xacro)
@@ -1,341 +1,10 @@
 <?xml version="1.0"?>
 <robot xmlns:xacro="http://www.ros.org/wiki/xacro">
-    <xacro:property name="hip_torque_max" value="200"/>
-    <xacro:property name="thigh_torque_max" value="200"/>
-    <xacro:property name="calf_torque_max" value="320"/>
-    <xacro:property name="ros_version" value="$(env ROS_VERSION)" />
-    <gazebo reference="imu_link">
-      <sensor name="imu_sensor" type="imu">
-      <plugin filename="libgazebo_ros_imu_sensor.so" name="imu_plugin">
-          <ros>
-            <namespace>/</namespace>
-            <remapping>~/out:=imu</remapping>
-          </ros>
-          <initial_orientation_as_reference>false</initial_orientation_as_reference>
-        </plugin>
-        <always_on>true</always_on>
-        <update_rate>100</update_rate>
-        <visualize>true</visualize>
-        <imu>
-          <angular_velocity>
-            <x>
-              <noise type="gaussian">
-                <mean>0.0</mean>
-                <stddev>0.0</stddev>
-                <bias_mean>0.0</bias_mean>
-                <bias_stddev>0.0</bias_stddev>
-              </noise>
-            </x>
-            <y>
-              <noise type="gaussian">
-                <mean>0.0</mean>
-                <stddev>0.0</stddev>
-                <bias_mean>0.0</bias_mean>
-                <bias_stddev>0.0</bias_stddev>
-              </noise>
-            </y>
-            <z>
-              <noise type="gaussian">
-                <mean>0.0</mean>
-                <stddev>0.0</stddev>
-                <bias_mean>0.0</bias_mean>
-                <bias_stddev>0.0</bias_stddev>
-              </noise>
-            </z>
-          </angular_velocity>
-          <linear_acceleration>
-            <x>
-              <noise type="gaussian">
-                <mean>0.0</mean>
-                <stddev>1.7e-2</stddev>
-                <bias_mean>0.1</bias_mean>
-                <bias_stddev>0.001</bias_stddev>
-              </noise>
-            </x>
-            <y>
-              <noise type="gaussian">
-                <mean>0.0</mean>
-                <stddev>1.7e-2</stddev>
-                <bias_mean>0.1</bias_mean>
-                <bias_stddev>0.001</bias_stddev>
-              </noise>
-            </y>
-            <z>
-              <noise type="gaussian">
-                <mean>0.0</mean>
-                <stddev>1.7e-2</stddev>
-                <bias_mean>0.1</bias_mean>
-                <bias_stddev>0.001</bias_stddev>
-              </noise>
-            </z>
-          </linear_acceleration>
-        </imu>
-      </sensor>
-    </gazebo>
-    <ros2_control name="GazeboSystem" type="system">
-        <hardware>
-            <plugin>gazebo_ros2_control/GazeboSystem</plugin>
-        </hardware>
-        <xacro:macro name="joint_interface" params="joint_name torque_limit">
-            <joint name="${joint_name}">
-            <command_interface name="effort">
-                <param name="min">-${torque_limit}</param>
-                <param name="max">${torque_limit}</param>
-            </command_interface>
-            <state_interface name="position"/>
-            <state_interface name="velocity"/>
-            <state_interface name="effort"/>
-            </joint>
-        </xacro:macro>
-        <xacro:macro name="leg_joints" params="prefix">
-            <xacro:joint_interface joint_name="${prefix}_hip_joint" torque_limit="${hip_torque_max}"/>
-            <xacro:joint_interface joint_name="${prefix}_thigh_joint" torque_limit="${thigh_torque_max}"/>
-            <xacro:joint_interface joint_name="${prefix}_calf_joint" torque_limit="${calf_torque_max}"/>
-        </xacro:macro>
-        <xacro:leg_joints prefix="FR"/>
-        <xacro:leg_joints prefix="FL"/>
-        <xacro:leg_joints prefix="RR"/>
-        <xacro:leg_joints prefix="RL"/>
-    </ros2_control>
-    <gazebo>
-        <plugin name="gazebo_ros2_control" filename="libgazebo_ros2_control.so">
-            <parameters>$(find b2_description)/config/robot_control_ros2.yaml</parameters>
-        </plugin>
-    </gazebo>
-    <gazebo reference="base">
-        <material>Gazebo/Green</material>
-        <turnGravityOff>false</turnGravityOff>
-    </gazebo>
-    <gazebo reference="trunk">
-        <mu1>0.2</mu1>
-        <mu2>0.2</mu2>
-        <kp  value="1000000.0"/>
-        <kd  value="1.0"/>
-    </gazebo>
-    <gazebo reference="stick_link">
-        <mu1>0.2</mu1>
-        <mu2>0.2</mu2>
-        <material>Gazebo/White</material>
-    </gazebo>
-    <gazebo reference="imu_link">
-        <mu1>0.2</mu1>
-        <mu2>0.2</mu2>
-        <material>Gazebo/Red</material>
-    </gazebo>
-    <!-- FL leg -->
-    <gazebo reference="FL_hip">
-        <mu1>0.2</mu1>
-        <mu2>0.2</mu2>
-        <!-- <material>Gazebo/DarkGrey</material> -->
-    </gazebo>
-    <gazebo reference="FL_thigh">
-        <mu1>0.2</mu1>
-        <mu2>0.2</mu2>
-        <self_collide>1</self_collide>
-        <!-- <material>Gazebo/DarkGrey</material> -->
-        <kp  value="1000000.0"/>
-        <kd  value="1.0"/>
-    </gazebo>
-    <gazebo reference="FL_calf">
-        <mu1>0.2</mu1>
-        <mu2>0.2</mu2>
-        <self_collide>1</self_collide>
-    </gazebo>
-    <gazebo reference="FL_foot">
-        <mu1>0.6</mu1>
-        <mu2>0.6</mu2>
-        <self_collide>1</self_collide>
-        <!-- <material>Gazebo/DarkGrey</material> -->
-        <kp  value="1000000.0"/>
-        <kd  value="1.0"/>
-    </gazebo>
-    <!-- FR leg -->
-    <gazebo reference="FR_hip">
-        <mu1>0.2</mu1>
-        <mu2>0.2</mu2>
-        <!-- <material>Gazebo/DarkGrey</material> -->
-    </gazebo>
-    <gazebo reference="FR_thigh">
-        <mu1>0.2</mu1>
-        <mu2>0.2</mu2>
-        <self_collide>1</self_collide>
-        <!-- <material>Gazebo/DarkGrey</material> -->
-        <kp  value="1000000.0"/>
-        <kd  value="1.0"/>
-    </gazebo>
-    <gazebo reference="FR_calf">
-        <mu1>0.2</mu1>
-        <mu2>0.2</mu2>
-        <self_collide>1</self_collide>
-    </gazebo>
-    <gazebo reference="FR_foot">
-        <mu1>0.6</mu1>
-        <mu2>0.6</mu2>
-        <self_collide>1</self_collide>
-        <!-- <material>Gazebo/DarkGrey</material> -->
-        <kp  value="1000000.0"/>
-        <kd  value="1.0"/>
-    </gazebo>
-    <!-- RL leg -->
-    <gazebo reference="RL_hip">
-        <mu1>0.2</mu1>
-        <mu2>0.2</mu2>
-        <!-- <material>Gazebo/DarkGrey</material> -->
-    </gazebo>
-    <gazebo reference="RL_thigh">
-        <mu1>0.2</mu1>
-        <mu2>0.2</mu2>
-        <self_collide>1</self_collide>
-        <!-- <material>Gazebo/DarkGrey</material> -->
-        <kp  value="1000000.0"/>
-        <kd  value="1.0"/>
-    </gazebo>
-    <gazebo reference="RL_calf">
-        <mu1>0.2</mu1>
-        <mu2>0.2</mu2>
-        <self_collide>1</self_collide>
-    </gazebo>
-    <gazebo reference="RL_foot">
-        <mu1>0.6</mu1>
-        <mu2>0.6</mu2>
-        <self_collide>1</self_collide>
-        <!-- <material>Gazebo/DarkGrey</material> -->
-        <kp  value="1000000.0"/>
-        <kd  value="1.0"/>
-    </gazebo>
-    <!-- RR leg -->
-    <gazebo reference="RR_hip">
-        <mu1>0.2</mu1>
-        <mu2>0.2</mu2>
-        <!-- <material>Gazebo/DarkGrey</material> -->
-    </gazebo>
-    <gazebo reference="RR_thigh">
-        <mu1>0.2</mu1>
-        <mu2>0.2</mu2>
-        <self_collide>1</self_collide>
-        <!-- <material>Gazebo/DarkGrey</material> -->
-        <kp  value="1000000.0"/>
-        <kd  value="1.0"/>
-    </gazebo>
-    <gazebo reference="RR_calf">
-        <mu1>0.2</mu1>
-        <mu2>0.2</mu2>
-        <self_collide>1</self_collide>
-    </gazebo>
-    <gazebo reference="RR_foot">
-        <mu1>0.6</mu1>
-        <mu2>0.6</mu2>
-        <self_collide>1</self_collide>
-        <!-- <material>Gazebo/DarkGrey</material> -->
-        <kp  value="1000000.0"/>
-        <kd  value="1.0"/>
-    </gazebo>
-    <gazebo reference="lidar_link">
-    <sensor name="lidar_3d" type="gpu_ray">
-        <update_rate>10</update_rate>
-        <visualize>false</visualize>
-        <ray>
-        <scan>
-            <!-- HORIZONTAL (360°) -->
-            <horizontal>
-            <samples>1800</samples>
-            <resolution>1</resolution>
-            <min_angle>-3.14159</min_angle>
-            <max_angle>3.14159</max_angle>
-            </horizontal>
-            <!-- VERTICAL (59°) -->
-            <vertical>
-            <samples>32</samples>
-            <resolution>1</resolution>
-            <min_angle>-0.9599</min_angle>   <!-- ~ -55° -->
-            <max_angle>0.2618</max_angle>    <!-- ~ +15° -->
-            </vertical>
-        </scan>
-        <range>
-            <min>0.07</min>
-            <max>100.0</max>
-            <resolution>0.01</resolution>
-        </range>
-        <noise>
-            <type>gaussian</type>
-            <mean>0.0</mean>
-            <stddev>0.007</stddev>
-        </noise>
-        </ray>
-        <!-- ROS 2 plugin -->
-        <plugin name="gazebo_ros_lidar" filename="libgazebo_ros_ray_sensor.so">
-        <ros>
-            <remapping>~/out:=rslidar_points</remapping>
-        </ros>
-        <frame_name>lidar_link</frame_name>
-        <output_type>sensor_msgs/PointCloud2</output_type>
-        </plugin>
-    </sensor>
-    </gazebo>
-    <gazebo reference="f_oc_link">
-    <sensor name="camera_sensor" type="camera">
-        <update_rate>30</update_rate>
-        <always_on>true</always_on>
-        <visualize>true</visualize>
-        <camera>
-        <horizontal_fov>1.396</horizontal_fov> <!-- ~120° -->
-        <image>
-            <width>1280</width>
-            <height>720</height>
-            <format>R8G8B8</format>
-        </image>
-        <clip>
-            <near>0.05</near>
-            <far>50.0</far>
-        </clip>
-        <!-- Optional noise -->
-        <noise>
-            <type>gaussian</type>
-            <mean>0.0</mean>
-            <stddev>0.01</stddev>
-        </noise>
-        </camera>
-        <plugin name="gazebo_ros_camera" filename="libgazebo_ros_camera.so">
-        <ros>
-            <namespace>/camera_front</namespace>
-            <remapping>~/image_raw:=image_raw</remapping>
-            <remapping>~/camera_info:=camera_info</remapping>
-        </ros>
-        <frame_name>f_oc_link</frame_name>
-        </plugin>
-    </sensor>
-    </gazebo>
-    <gazebo reference="r_oc_link">
-    <sensor name="camera_sensor" type="camera">
-        <update_rate>30</update_rate>
-        <always_on>true</always_on>
-        <visualize>true</visualize>
-        <camera>
-        <horizontal_fov>1.396</horizontal_fov> <!-- ~120° -->
-        <image>
-            <width>1280</width>
-            <height>720</height>
-            <format>R8G8B8</format>
-        </image>
-        <clip>
-            <near>0.05</near>
-            <far>50.0</far>
-        </clip>
-        <!-- Optional noise -->
-        <noise>
-            <type>gaussian</type>
-            <mean>0.0</mean>
-            <stddev>0.01</stddev>
-        </noise>
-        </camera>
-        <plugin name="gazebo_ros_camera" filename="libgazebo_ros_camera.so">
-        <ros>
-            <namespace>/camera_back</namespace>
-            <remapping>~/image_raw:=image_raw</remapping>
-            <remapping>~/camera_info:=camera_info</remapping>
-        </ros>
-        <frame_name>r_oc_link</frame_name>
-        </plugin>
-    </sensor>
-    </gazebo>
+    <xacro:include filename="$(find b2_description)/xacro/properties.xacro"/>
+    <xacro:include filename="$(find b2_description)/xacro/sensors/imu.xacro"/>
+    <xacro:include filename="$(find b2_description)/xacro/sensors/lidar.xacro"/>
+    <xacro:include filename="$(find b2_description)/xacro/sensors/camera.xacro"/>
+    <xacro:include filename="$(find b2_description)/xacro/control/ros2_control.xacro"/>
+    <xacro:include filename="$(find b2_description)/xacro/materials/body.xacro"/>
+    <xacro:include filename="$(find b2_description)/xacro/materials/legs.xacro"/>
 </robot>

File: src/b2_description/xacro/robot.xacro (robot description, xacro)
@@ -1,4 +1,5 @@
 <?xml version="1.0"?>
 <robot name="b2_description" xmlns:xacro="http://www.ros.org/wiki/xacro">
+    <xacro:arg name="gpu" default="true"/>
     <xacro:include filename="$(find b2_description)/urdf/b2_description.urdf"/>
     <xacro:include filename="$(find b2_description)/xacro/gazebo.xacro"/>
