Commit message: update for our env

File: src/b2_description/urdf/b2_description.urdf (robot description, URDF)
Before this commit: robot b2_description, 37 links, 36 joints
Joints:
- joint joint_f_oc: origin xyz=0.39079 0 -0.013433 rpy=-1.5708 0 -1.5708 -> xyz=0.39079 0 -0.013433 rpy=0 0 0
- joint joint_r_oc: origin xyz=-0.38451 0 -0.023249 rpy=-1.5708 0 1.5708 -> xyz=-0.38451 0 -0.023249 rpy=0 0 3.14159

File: src/b2_description/xacro/gazebo.xacro (robot description, xacro)
@@ -5,127 +5,4 @@
     <xacro:property name="calf_torque_max" value="320"/>
     <xacro:property name="ros_version" value="$(env ROS_VERSION)" />
-    <xacro:if value="${int(ros_version) == 1}">
-    <!-- ros_control plugin -->
-    <gazebo>
-        <plugin name="gazebo_ros_control" filename="libgazebo_ros_control.so">
-            <robotNamespace>/b2_gazebo</robotNamespace>
-            <robotSimType>gazebo_ros_control/DefaultRobotHWSim</robotSimType>
-        </plugin>
-    </gazebo>
-    <!-- Show the trajectory of trunk center. -->
-    <!-- <gazebo>
-        <plugin name="3dplot" filename="libLinkPlot3DPlugin.so">
-            <frequency>10</frequency>
-            <plot>
-                <link>base</link>
-                <pose>0 0 0 0 0 0</pose>
-                <material>Gazebo/Yellow</material>
-            </plot>
-        </plugin>
-    </gazebo> -->
-    <!-- Show the trajectory of foot. You can add another trajectory about another foot. -->
-    <!-- <gazebo>
-        <plugin name="3dplot" filename="libLinkPlot3DPlugin.so">
-            <frequency>100</frequency>
-            <plot>
-                <link>FL_foot</link>
-                <pose>0 0 0 0 0 0</pose>
-                <material>Gazebo/Green</material>
-            </plot>
-        </plugin>
-    </gazebo> -->
-    <gazebo>
-        <plugin filename="libgazebo_ros_force.so" name="gazebo_ros_force">
-            <bodyName>trunk</bodyName>
-            <topicName>/apply_force/trunk</topicName>
-        </plugin>
-    </gazebo>
-    <gazebo reference="imu_link">
-        <gravity>true</gravity>
-        <sensor name="imu_sensor" type="imu">
-            <always_on>true</always_on>
-            <update_rate>1000</update_rate>
-            <visualize>true</visualize>
-            <topic>__default_topic__</topic>
-            <plugin filename="libgazebo_ros_imu_sensor.so" name="imu_plugin">
-                <topicName>trunk_imu</topicName>
-                <bodyName>imu_link</bodyName>
-                <updateRateHZ>1000.0</updateRateHZ>
-                <gaussianNoise>0.0</gaussianNoise>
-                <xyzOffset>0 0 0</xyzOffset>
-                <rpyOffset>0 0 0</rpyOffset>
-                <frameName>imu_link</frameName>
-            </plugin>
-            <pose>0 0 0 0 0 0</pose>
-        </sensor>
-    </gazebo>
-    <!-- Foot contacts. -->
-    <gazebo reference="FR_calf">
-        <sensor name="FR_foot_contact" type="contact">
-        <update_rate>100</update_rate>
-        <plugin name="contactPlugin" filename="libunitreeFootContactPlugin.so"/>
-        <contact>
-            <collision>FR_calf_fixed_joint_lump__FR_foot_collision_1</collision>
-        </contact>
-        </sensor>
-    </gazebo>
-    <gazebo reference="FL_calf">
-        <sensor name="FL_foot_contact" type="contact">
-        <update_rate>100</update_rate>
-        <plugin name="contactPlugin" filename="libunitreeFootContactPlugin.so"/>
-        <contact>
-            <collision>FL_calf_fixed_joint_lump__FL_foot_collision_1</collision>
-        </contact>
-        </sensor>
-    </gazebo>
-    <gazebo reference="RR_calf">
-        <sensor name="RR_foot_contact" type="contact">
-        <update_rate>100</update_rate>
-        <plugin name="contactPlugin" filename="libunitreeFootContactPlugin.so"/>
-        <contact>
-            <collision>RR_calf_fixed_joint_lump__RR_foot_collision_1</collision>
-        </contact>
-        </sensor>
-    </gazebo>
-    <gazebo reference="RL_calf">
-        <sensor name="RL_foot_contact" type="contact">
-        <update_rate>100</update_rate>
-        <plugin name="contactPlugin" filename="libunitreeFootContactPlugin.so"/>
-        <contact>
-            <collision>RL_calf_fixed_joint_lump__RL_foot_collision_1</collision>
-        </contact>
-        </sensor>
-    </gazebo>
-    <!-- Visualization of Foot contacts. -->
-    <!-- <gazebo reference="FR_foot">
-        <visual>
-            <plugin name="drawForcePlugin" filename="libunitreeDrawForcePlugin.so">
-                <topicName>FR_foot_contact</topicName>
-            </plugin>
-        </visual>
-    </gazebo>
-    <gazebo reference="FL_foot">
-        <visual>
-            <plugin name="drawForcePlugin" filename="libunitreeDrawForcePlugin.so">
-                <topicName>FL_foot_contact</topicName>
-            </plugin>
-        </visual>
-    </gazebo>
-    <gazebo reference="RR_foot">
-        <visual>
-            <plugin name="drawForcePlugin" filename="libunitreeDrawForcePlugin.so">
-                <topicName>RR_foot_contact</topicName>
-            </plugin>
-        </visual>
-    </gazebo>
-    <gazebo reference="RL_foot">
-        <visual>
-            <plugin name="drawForcePlugin" filename="libunitreeDrawForcePlugin.so">
-                <topicName>RL_foot_contact</topicName>
-            </plugin>
-        </visual>
-    </gazebo> -->
-    </xacro:if>
-    <xacro:if value="${int(ros_version) == 2}">
     <gazebo reference="imu_link">
       <sensor name="imu_sensor" type="imu">
@@ -145,7 +22,7 @@
               <noise type="gaussian">
                 <mean>0.0</mean>
-                <stddev>2e-4</stddev>
-                <bias_mean>0.0000075</bias_mean>
-                <bias_stddev>0.0000008</bias_stddev>
+                <stddev>0.0</stddev>
+                <bias_mean>0.0</bias_mean>
+                <bias_stddev>0.0</bias_stddev>
               </noise>
             </x>
@@ -153,7 +30,7 @@
               <noise type="gaussian">
                 <mean>0.0</mean>
-                <stddev>2e-4</stddev>
-                <bias_mean>0.0000075</bias_mean>
-                <bias_stddev>0.0000008</bias_stddev>
+                <stddev>0.0</stddev>
+                <bias_mean>0.0</bias_mean>
+                <bias_stddev>0.0</bias_stddev>
               </noise>
             </y>
@@ -161,7 +38,7 @@
               <noise type="gaussian">
                 <mean>0.0</mean>
-                <stddev>2e-4</stddev>
-                <bias_mean>0.0000075</bias_mean>
-                <bias_stddev>0.0000008</bias_stddev>
+                <stddev>0.0</stddev>
+                <bias_mean>0.0</bias_mean>
+                <bias_stddev>0.0</bias_stddev>
               </noise>
             </z>
@@ -226,5 +103,4 @@
         </plugin>
     </gazebo>
-    </xacro:if>
     <gazebo reference="base">
         <material>Gazebo/Green</material>
@@ -355,3 +231,111 @@
         <kd  value="1.0"/>
     </gazebo>
+    <gazebo reference="lidar_link">
+    <sensor name="lidar_3d" type="gpu_ray">
+        <update_rate>10</update_rate>
+        <visualize>false</visualize>
+        <ray>
+        <scan>
+            <!-- HORIZONTAL (360°) -->
+            <horizontal>
+            <samples>1800</samples>
+            <resolution>1</resolution>
+            <min_angle>-3.14159</min_angle>
+            <max_angle>3.14159</max_angle>
+            </horizontal>
+            <!-- VERTICAL (59°) -->
+            <vertical>
+            <samples>32</samples>
+            <resolution>1</resolution>
+            <min_angle>-0.9599</min_angle>   <!-- ~ -55° -->
+            <max_angle>0.2618</max_angle>    <!-- ~ +15° -->
+            </vertical>
+        </scan>
+        <range>
+            <min>0.07</min>
+            <max>100.0</max>
+            <resolution>0.01</resolution>
+        </range>
+        <noise>
+            <type>gaussian</type>
+            <mean>0.0</mean>
+            <stddev>0.007</stddev>
+        </noise>
+        </ray>
+        <!-- ROS 2 plugin -->
+        <plugin name="gazebo_ros_lidar" filename="libgazebo_ros_ray_sensor.so">
+        <ros>
+            <remapping>~/out:=rslidar_points</remapping>
+        </ros>
+        <frame_name>lidar_link</frame_name>
+        <output_type>sensor_msgs/PointCloud2</output_type>
+        </plugin>
+    </sensor>
+    </gazebo>
+    <gazebo reference="f_oc_link">
+    <sensor name="camera_sensor" type="camera">
+        <update_rate>30</update_rate>
+        <always_on>true</always_on>
+        <visualize>true</visualize>
+        <camera>
+        <horizontal_fov>1.396</horizontal_fov> <!-- ~120° -->
+        <image>
+            <width>1280</width>
+            <height>720</height>
+            <format>R8G8B8</format>
+        </image>
+        <clip>
+            <near>0.05</near>
+            <far>50.0</far>
+        </clip>
+        <!-- Optional noise -->
+        <noise>
+            <type>gaussian</type>
+            <mean>0.0</mean>
+            <stddev>0.01</stddev>
+        </noise>
+        </camera>
+        <plugin name="gazebo_ros_camera" filename="libgazebo_ros_camera.so">
+        <ros>
+            <namespace>/camera_front</namespace>
+            <remapping>~/image_raw:=image_raw</remapping>
+            <remapping>~/camera_info:=camera_info</remapping>
+        </ros>
+        <frame_name>f_oc_link</frame_name>
+        </plugin>
+    </sensor>
+    </gazebo>
+    <gazebo reference="r_oc_link">
+    <sensor name="camera_sensor" type="camera">
+        <update_rate>30</update_rate>
+        <always_on>true</always_on>
+        <visualize>true</visualize>
+        <camera>
+        <horizontal_fov>1.396</horizontal_fov> <!-- ~120° -->
+        <image>
+            <width>1280</width>
+            <height>720</height>
+            <format>R8G8B8</format>
+        </image>
+        <clip>
+            <near>0.05</near>
+            <far>50.0</far>
+        </clip>
+        <!-- Optional noise -->
+        <noise>
+            <type>gaussian</type>
+            <mean>0.0</mean>
+            <stddev>0.01</stddev>
+        </noise>
+        </camera>
+        <plugin name="gazebo_ros_camera" filename="libgazebo_ros_camera.so">
+        <ros>
+            <namespace>/camera_back</namespace>
+            <remapping>~/image_raw:=image_raw</remapping>
+            <remapping>~/camera_info:=camera_info</remapping>
+        </ros>
+        <frame_name>r_oc_link</frame_name>
+        </plugin>
+    </sensor>
+    </gazebo>
 </robot>

Commit message: add third view camera

File: src/b2_description/urdf/b2_description.urdf (robot description, URDF)
Before this commit: robot b2_description, 37 links, 36 joints
Links:
- added link tb_oc_link, mass 4.19E-15
- added link tf_oc_link, mass 4.19E-12
Joints:
- added joint joint_tb_oc: type fixed, parent base_link, child tb_oc_link, origin xyz=-1.39079 0 0.5 rpy=0 0.349066 0, axis 0 0 0
- added joint joint_tf_oc: type fixed, parent base_link, child tf_oc_link, origin xyz=1.3 0 0.5 rpy=0 0.349066 3.14159, axis 0 0 0

File: src/b2_description/xacro/sensors/camera.xacro (robot description, xacro)
@@ -37,3 +37,5 @@
     <xacro:camera_sensor link_name="f_oc_link" namespace="/camera_front"/>
     <xacro:camera_sensor link_name="r_oc_link" namespace="/camera_back"/>
+    <xacro:camera_sensor link_name="tf_oc_link" namespace="/camera_third_front"/>
+    <xacro:camera_sensor link_name="tb_oc_link" namespace="/camera_third_back"/>
 </robot>
