Commit message: update robot joint initial value

File: src/b2_description/xacro/control/ros2_control.xacro (robot description, xacro)
@@ -5,5 +5,5 @@
             <plugin>gazebo_ros2_control/GazeboSystem</plugin>
         </hardware>
-        <xacro:macro name="joint_interface" params="joint_name torque_limit">
+        <xacro:macro name="joint_interface" params="joint_name torque_limit initial_position">
             <joint name="${joint_name}">
                 <command_interface name="effort">
@@ -11,5 +11,7 @@
                     <param name="max">${torque_limit}</param>
                 </command_interface>
-                <state_interface name="position"/>
+                <state_interface name="position">
+                    <param name="initial_value">${initial_position}</param>
+                </state_interface>
                 <state_interface name="velocity"/>
                 <state_interface name="effort"/>
@@ -17,7 +19,7 @@
         </xacro:macro>
         <xacro:macro name="leg_joints" params="prefix">
-            <xacro:joint_interface joint_name="${prefix}_hip_joint" torque_limit="${hip_torque_max}"/>
-            <xacro:joint_interface joint_name="${prefix}_thigh_joint" torque_limit="${thigh_torque_max}"/>
-            <xacro:joint_interface joint_name="${prefix}_calf_joint" torque_limit="${calf_torque_max}"/>
+            <xacro:joint_interface joint_name="${prefix}_hip_joint" torque_limit="${hip_torque_max}" initial_position="${default_hip_pos}"/>
+            <xacro:joint_interface joint_name="${prefix}_thigh_joint" torque_limit="${thigh_torque_max}" initial_position="${default_thigh_pos}"/>
+            <xacro:joint_interface joint_name="${prefix}_calf_joint" torque_limit="${calf_torque_max}" initial_position="${default_calf_pos}"/>
         </xacro:macro>
         <xacro:leg_joints prefix="FR"/>

File: src/b2_description/xacro/properties.xacro (robot description, xacro)
@@ -4,4 +4,8 @@
     <xacro:property name="thigh_torque_max" value="200"/>
     <xacro:property name="calf_torque_max" value="320"/>
+    <!-- Folded leg pose from mjcf/b2.xml home keyframe -->
+    <xacro:property name="default_hip_pos" value="0.0"/>
+    <xacro:property name="default_thigh_pos" value="1.28"/>
+    <xacro:property name="default_calf_pos" value="-2.84"/>
     <xacro:property name="ros_version" value="$(env ROS_VERSION)" />
 </robot>
